Commit message: fix: Replace OGRE specific colors with modern Gazebo color definitions.

File: ora_description/description/anteater_core.xacro (robot description, xacro)
@@ -41,5 +41,9 @@
   </link>
   <gazebo reference="chassis_link">
-    <material>Gazebo/White</material>
+    <material>
+      <ambient>1 1 1 1</ambient>
+      <diffuse>1 1 1 1</diffuse>
+      <specular>0.5 0.5 0.5 1</specular>
+    </material>
   </gazebo>
 </robot>

File: ora_description/description/caster.xacro (robot description, xacro)
@@ -31,5 +31,9 @@
     </joint>
     <gazebo reference="${prefix}_front_caster_link">
-      <material>Gazebo/Black</material>
+      <material>
+        <ambient>0.1 0.1 0.1 1</ambient>
+        <diffuse>0.1 0.1 0.1 1</diffuse>
+        <specular>0.5 0.5 0.5 1</specular>
+      </material>
       <!-- Frictionless-ish -->
       <!-- Stops the robot from jumping around -->
@@ -66,5 +70,9 @@
     </joint>
     <gazebo reference="${prefix}_back_caster_link">
-      <material>Gazebo/Black</material>
+      <material>
+        <ambient>0.1 0.1 0.1 1</ambient>
+        <diffuse>0.1 0.1 0.1 1</diffuse>
+        <specular>0.5 0.5 0.5 1</specular>
+      </material>
       <!-- Frictionless-ish -->
       <!-- Stops the robot from jumping around -->

File: ora_description/description/wheel.xacro (robot description, xacro)
@@ -27,5 +27,9 @@
     </link>
     <gazebo reference="${prefix}_wheel_link">
-      <material>Gazebo/Black</material>
+      <material>
+        <ambient>0.1 0.1 0.1 1</ambient>
+        <diffuse>0.1 0.1 0.1 1</diffuse>
+        <specular>0.5 0.5 0.5 1</specular>
+      </material>
     </gazebo>
   </xacro:macro>

Commit message: fix: Switch URDF files to colors defined in the materials.xacro file.

File: ora_description/description/anteater_core.xacro (robot description, xacro)
@@ -41,9 +41,5 @@
   </link>
   <gazebo reference="chassis_link">
-    <material>
-      <ambient>1 1 1 1</ambient>
-      <diffuse>1 1 1 1</diffuse>
-      <specular>0.5 0.5 0.5 1</specular>
-    </material>
+    <material name="white"/>
   </gazebo>
 </robot>

File: ora_description/description/caster.xacro (robot description, xacro)
@@ -13,5 +13,5 @@
           <cylinder radius="${front_caster_radius}" length="${front_caster_width}"/>
         </geometry>
-        <material name="gray"/>
+        <material name="black"/>
       </visual>
       <collision>
@@ -31,13 +31,9 @@
     </joint>
     <gazebo reference="${prefix}_front_caster_link">
-      <material>
-        <ambient>0.1 0.1 0.1 1</ambient>
-        <diffuse>0.1 0.1 0.1 1</diffuse>
-        <specular>0.5 0.5 0.5 1</specular>
-      </material>
+      <material name="black"/>
       <!-- Frictionless-ish -->
       <!-- Stops the robot from jumping around -->
-      <mu1 value="0.001"/>
-      <mu2 value="0.001"/>
+      <mu1>0.001</mu1>
+      <mu2>0.001</mu2>
     </gazebo>
   </xacro:macro>
@@ -52,5 +48,5 @@
           <cylinder radius="${back_caster_radius}" length="${back_caster_width}"/>
         </geometry>
-        <material name="gray"/>
+        <material name="black"/>
       </visual>
       <collision>
@@ -70,13 +66,9 @@
     </joint>
     <gazebo reference="${prefix}_back_caster_link">
-      <material>
-        <ambient>0.1 0.1 0.1 1</ambient>
-        <diffuse>0.1 0.1 0.1 1</diffuse>
-        <specular>0.5 0.5 0.5 1</specular>
-      </material>
+      <material name="black"/>
       <!-- Frictionless-ish -->
       <!-- Stops the robot from jumping around -->
-      <mu1 value="0.001"/>
-      <mu2 value="0.001"/>
+      <mu1>0.001</mu1>
+      <mu2>0.001</mu2>
     </gazebo>
   </xacro:macro>

File: ora_description/description/wheel.xacro (robot description, xacro)
@@ -27,9 +27,5 @@
     </link>
     <gazebo reference="${prefix}_wheel_link">
-      <material>
-        <ambient>0.1 0.1 0.1 1</ambient>
-        <diffuse>0.1 0.1 0.1 1</diffuse>
-        <specular>0.5 0.5 0.5 1</specular>
-      </material>
+      <material name="black"/>
     </gazebo>
   </xacro:macro>

Commit message: add sesnor tower

File: ora_description/description/anteater_core.xacro (robot description, xacro)
@@ -43,3 +43,30 @@
     <material name="white"/>
   </gazebo>
+  <!-- TOWER LINK -->
+  <joint name="tower_joint" type="fixed">
+    <parent link="chassis_link"/>
+    <child link="tower_link"/>
+    <origin xyz="${tower_x_offset} 0 ${(base_z_offset / 2) + tower_z_offset}" rpy="0 0 0"/>
+  </joint>
+  <link name="tower_link">
+    <visual>
+      <origin xyz="0 0 0" rpy="0 0 0"/>
+      <geometry>
+        <box size="${tower_length} ${tower_width} ${tower_height}"/>
+      </geometry>
+      <material name="white"/>
+    </visual>
+    <collision>
+      <origin xyz="0 0 0" rpy="0 0 0"/>
+      <geometry>
+        <box size="${tower_length} ${tower_width} ${tower_height}"/>
+      </geometry>
+    </collision>
+    <xacro:inertial_box mass="5.0" x="${tower_length}" y="${tower_width}" z="${tower_height}">
+      <origin xyz="0 0 0" rpy="0 0 0"/>
+    </xacro:inertial_box>
+  </link>
+  <gazebo reference="tower_link">
+    <material name="white"/>
+  </gazebo>
 </robot>

File: ora_description/description/dimensions.xacro (robot description, xacro)
@@ -14,4 +14,8 @@
   <xacro:property name="base_width" value="${29.45 * in_to_m}"/>
   <xacro:property name="base_height" value="${18.75 * in_to_m}"/>
+  <!-- Tower Dimensions -->
+  <xacro:property name="tower_length" value="${0.75 * in_to_m}"/>
+  <xacro:property name="tower_width" value="${8.625 * in_to_m}"/>
+  <xacro:property name="tower_height" value="${26.25 * in_to_m}"/>
   <!-- Wheel Dimensions / Location -->
   <xacro:property name="main_wheel_diameter" value="${11.97 * in_to_m}"/>
@@ -44,4 +48,6 @@
   <xacro:property name="base_x_offset" value="${(back_caster_x_offset / 4)}"/>
   <xacro:property name="base_z_offset" value="${7.375 * in_to_m}"/>
+  <xacro:property name="tower_x_offset" value="${(-base_length / 2) + base_x_offset + (tower_length / 2) + (12.75 * in_to_m)}"/>
+  <xacro:property name="tower_z_offset" value="${base_height + base_z_offset}"/>
   <xacro:property name="lidar_x_offset" value="${(base_length / 2) - (lidar_radius / 2) + (base_x_offset / 2)}"/>
   <xacro:property name="lidar_z_offset" value="${(base_height / 2) + (lidar_height / 2) + base_z_offset}"/>
