Commit message: updated robot's dimensions

File: ora_description/description/dimensions.xacro (robot description, xacro)
@@ -3,4 +3,6 @@
   <!-- This file contains the dimensions of the robot -->
   <!-- The dimensions are defined in meters -->
+  <!-- Real robot dimensions -->
+  <!-- https://discord.com/channels/690363866437386281/879501498004946944/1508609648339583047 -->
   <!-- Convert mm to meters -->
   <xacro:property name="mm_to_m" value="${0.001}"/>
@@ -9,13 +11,13 @@
   <xacro:property name="in_to_m" value="${0.0254}"/>
   <!-- Base Chassis Dimensions -->
-  <xacro:property name="base_length" value="${34 * in_to_m}"/>
-  <xacro:property name="base_width" value="${17.5 * in_to_m}"/>
-  <xacro:property name="base_height" value="${10 * in_to_m}"/>
+  <xacro:property name="base_length" value="${45.5 * in_to_m}"/>
+  <xacro:property name="base_width" value="${29.45 * in_to_m}"/>
+  <xacro:property name="base_height" value="${18.75 * in_to_m}"/>
   <!-- Wheel Dimensions / Location -->
-  <xacro:property name="main_wheel_diameter" value="${33.02 * cm_to_m}"/>
+  <xacro:property name="main_wheel_diameter" value="${11.97 * in_to_m}"/>
   <xacro:property name="main_wheel_radius" value="${main_wheel_diameter / 2}"/>
   <xacro:property name="main_wheel_width" value="${48 * mm_to_m}"/>
   <xacro:property name="main_wheel_z_offset" value="${0.0}"/>
-  <xacro:property name="main_wheel_y_offset" value="${28.575 * cm_to_m}"/>
+  <xacro:property name="main_wheel_y_offset" value="${((23.93 * in_to_m) - main_wheel_width) / 2}"/>
   <xacro:property name="main_wheel_x_offset" value="${0.0}"/>
   <!-- Caster Dimensions / Location -->
@@ -38,7 +40,8 @@
   <xacro:property name="gps_height" value="${20 * mm_to_m}"/>
   <xacro:property name="gps_radius" value="${50 * mm_to_m / 2}"/>
+  <!-- TODO add IMU dimensions and offsets -->
   <!-- Assorted Offset Values -->
   <xacro:property name="base_x_offset" value="${(back_caster_x_offset / 4)}"/>
-  <xacro:property name="base_z_offset" value="${back_caster_radius / 4}"/>
+  <xacro:property name="base_z_offset" value="${7.375 * in_to_m}"/>
   <xacro:property name="lidar_x_offset" value="${(base_length / 2) - (lidar_radius / 2) + (base_x_offset / 2)}"/>
   <xacro:property name="lidar_z_offset" value="${(base_height / 2) + (lidar_height / 2) + base_z_offset}"/>

Commit message: update sensors to real positions

File: ora_description/description/dimensions.xacro (robot description, xacro)
@@ -42,6 +42,10 @@
   <xacro:property name="lidar_radius" value="${103.3 * mm_to_m / 2}"/>
   <!-- GPS Dimensions -->
-  <xacro:property name="gps_height" value="${20 * mm_to_m}"/>
-  <xacro:property name="gps_radius" value="${50 * mm_to_m / 2}"/>
+  <xacro:property name="gps_height" value="${0.875 * in_to_m}"/>
+  <xacro:property name="gps_radius" value="${2.5 * in_to_m / 2}"/>
+  <!-- Camera Dimensions -->
+  <xacro:property name="camera_length" value="0.015"/>
+  <xacro:property name="camera_width" value="0.130"/>
+  <xacro:property name="camera_height" value="0.022"/>
   <!-- TODO add IMU dimensions and offsets -->
   <!-- Assorted Offset Values -->
@@ -50,7 +54,9 @@
   <xacro:property name="tower_x_offset" value="${(-base_length / 2) + base_x_offset + (tower_length / 2) + (12.75 * in_to_m)}"/>
   <xacro:property name="tower_z_offset" value="${base_height + base_z_offset}"/>
-  <xacro:property name="lidar_x_offset" value="${(base_length / 2) - (lidar_radius / 2) + (base_x_offset / 2)}"/>
-  <xacro:property name="lidar_z_offset" value="${(base_height / 2) + (lidar_height / 2) + base_z_offset}"/>
-  <xacro:property name="gps_x_offset" value="${0}"/>
-  <xacro:property name="gps_z_offset" value="${(base_height / 2) + (gps_height / 2) + base_z_offset}"/>
+  <xacro:property name="lidar_x_offset" value="${28.49 * in_to_m}"/>
+  <xacro:property name="lidar_z_offset" value="${4.62 * in_to_m}"/>
+  <xacro:property name="gps_x_offset" value="${tower_x_offset}"/>
+  <xacro:property name="gps_z_offset" value="${(tower_height / 2) + (gps_height / 2)}"/>
+  <xacro:property name="camera_x_offset" value="${(tower_length / 2) + (2 * in_to_m)}"/>
+  <xacro:property name="camera_z_offset" value="${(tower_height / 2)}"/>
 </robot>

File: ora_description/description/sensors.xacro (robot description, xacro)
@@ -5,9 +5,7 @@
   <!-- Lidar -->
   <link name="lidar_link">
-    <inertial>
-      <origin xyz="0 0 0" rpy="0 0 0"/>
-      <mass value="0.125"/>
-      <inertia ixx="0.001" ixy="0" ixz="0" iyy="0.001" iyz="0" izz="0.001" />
-    </inertial>
+    <xacro:inertial_cylinder mass="0.125" length="${lidar_height}" radius="${lidar_radius}">
+      <origin xyz="0 0 0" rpy="0 0 0"/>
+    </xacro:inertial_cylinder>
     <collision>
       <origin xyz="0 0 0" rpy="0 0 0"/>
@@ -21,5 +19,5 @@
         <cylinder radius="${lidar_radius}" length="${lidar_height}"/>
       </geometry>
-      <material name="dark_gray"/>
+      <material name="blue"/>
     </visual>
   </link>
@@ -29,4 +27,11 @@
     <origin xyz="${lidar_x_offset} 0 ${lidar_z_offset}" rpy="0 0 0"/>
   </joint>
+  <xacro:unless value="$(arg sim_mode)">
+    <joint name="velodyne_joint" type="fixed">
+      <parent link="lidar_link"/>
+      <child link="velodyne"/>
+      <origin xyz="0 0 0" rpy="0 0 0"/>
+    </joint>
+  </xacro:unless>
   <!-- Lidar Plugin -->
   <gazebo reference="lidar_link">
@@ -71,24 +76,22 @@
       <origin xyz="0 0 0" rpy="0 0 0"/>
       <geometry>
-        <box size="0.015 0.130 0.022"/>
-      </geometry>
-      <material name="dark_gray"/>
-    </visual>
-    <collision>
-      <origin xyz="0 0 0" rpy="0 0 0"/>
-      <geometry>
-        <box size="0.015 0.130 0.022"/>
-      </geometry>
-    </collision>
-    <inertial>
-      <origin xyz="0 0 0" rpy="0 0 0"/>
-      <mass value="0.035"/>
-      <inertia ixx="0.001" ixy="0" ixz="0" iyy="0.001" iyz="0" izz="0.001" />
-    </inertial>
+        <box size="${camera_length} ${camera_width} ${camera_height}"/>
+      </geometry>
+      <material name="yellow"/>
+    </visual>
+    <collision>
+      <origin xyz="0 0 0" rpy="0 0 0"/>
+      <geometry>
+        <box size="${camera_length} ${camera_width} ${camera_height}"/>
+      </geometry>
+    </collision>
+    <xacro:inertial_box mass="0.035" x="${camera_length}" y="${camera_width}" z="${camera_height}">
+      <origin xyz="0 0 0" rpy="0 0 0"/>
+    </xacro:inertial_box>
   </link>
   <joint name="camera_joint" type="fixed">
-    <parent link="base_link"/>
+    <parent link="tower_link"/>
     <child link="camera_link"/>
-    <origin xyz="0.2 0 0.4" rpy="0 0 0"/>
+    <origin xyz="${camera_x_offset} 0 ${camera_z_offset}" rpy="0 0.610865 0"/>
   </joint>
   <!-- For use with the line detection -->
@@ -135,9 +138,7 @@
   <!-- GPS -->
   <link name="gnss_link">
-    <inertial>
-      <origin xyz="0 0 0" rpy="0 0 0"/>
-      <mass value="0.125"/>
-      <inertia ixx="0.001" ixy="0" ixz="0" iyy="0.001" iyz="0" izz="0.001" />
-    </inertial>
+    <xacro:inertial_cylinder mass="0.125" length="${gps_height}" radius="${gps_radius}">
+      <origin xyz="0 0 0" rpy="0 0 0"/>
+    </xacro:inertial_cylinder>
     <collision>
       <origin xyz="0 0 0" rpy="0 0 0"/>
@@ -151,11 +152,11 @@
         <cylinder radius="${gps_radius}" length="${gps_height}"/>
       </geometry>
-      <material name="dark_gray"/>
+      <material name="red"/>
     </visual>
   </link>
   <joint name="gps_joint" type="fixed">
-    <parent link="base_link"/>
+    <parent link="tower_link"/>
     <child link="gnss_link"/>
-    <origin xyz="${gps_x_offset} 0 ${gps_z_offset}" rpy="0 0 0"/>
+    <origin xyz="0 0 ${gps_z_offset}" rpy="0 0 0"/>
   </joint>
   <!-- <gazebo reference="gnss_link">

Commit message: update IMU to real

File: ora_description/description/dimensions.xacro (robot description, xacro)
@@ -48,5 +48,8 @@
   <xacro:property name="camera_width" value="0.130"/>
   <xacro:property name="camera_height" value="0.022"/>
-  <!-- TODO add IMU dimensions and offsets -->
+  <!-- IMU Dimensions -->
+  <xacro:property name="imu_length" value="${25 * mm_to_m}"/>
+  <xacro:property name="imu_width" value="${15 * mm_to_m}"/>
+  <xacro:property name="imu_height" value="${10 * mm_to_m}"/>
   <!-- Assorted Offset Values -->
   <xacro:property name="base_x_offset" value="${(back_caster_x_offset / 4)}"/>
@@ -60,3 +63,4 @@
   <xacro:property name="camera_x_offset" value="${(tower_length / 2) + (2 * in_to_m)}"/>
   <xacro:property name="camera_z_offset" value="${(tower_height / 2)}"/>
+  <xacro:property name="imu_z_offset" value="${base_z_offset + (base_height / 2) - (0.25 * in_to_m)}"/>
 </robot>

File: ora_description/description/sensors.xacro (robot description, xacro)
@@ -186,20 +186,18 @@
   <!-- IMU -->
   <link name="imu_link">
-    <inertial>
-      <origin xyz="0 0 0" rpy="0 0 0"/>
-      <mass value="0.1"/>
-      <inertia ixx="0.0001" ixy="0" ixz="0" iyy="0.0001" iyz="0" izz="0.0001"/>
-    </inertial>
-    <visual>
-      <origin xyz="0 0 0" rpy="0 0 0"/>
-      <geometry>
-        <box size="0.1 0.1 0.1"/>
-      </geometry>
-      <material name="dark_gray"/>
-    </visual>
-    <collision>
-      <origin xyz="0 0 0" rpy="0 0 0"/>
-      <geometry>
-        <box size="0.1 0.1 0.1"/>
+    <xacro:inertial_box mass="0.01" x="${imu_length}" y="${imu_width}" z="${imu_height}">
+      <origin xyz="0 0 0" rpy="0 0 0"/>
+    </xacro:inertial_box>
+    <visual>
+      <origin xyz="0 0 0" rpy="0 0 0"/>
+      <geometry>
+        <box size="${imu_length} ${imu_width} ${imu_height}"/>
+      </geometry>
+      <material name="purple"/>
+    </visual>
+    <collision>
+      <origin xyz="0 0 0" rpy="0 0 0"/>
+      <geometry>
+        <box size="${imu_length} ${imu_width} ${imu_height}"/>
       </geometry>
     </collision>
@@ -208,5 +206,5 @@
     <parent link="base_link"/>
     <child link="imu_link"/>
-    <origin xyz="0 0 0.01" rpy="0 0 0"/>
+    <origin xyz="0 0 ${imu_z_offset}" rpy="0 0 0"/>
   </joint>
   <!-- IMU Plugin -->

Commit message: Adjust GPS offset

File: ora_description/description/dimensions.xacro (robot description, xacro)
@@ -59,5 +59,6 @@
   <xacro:property name="lidar_x_offset" value="${28.49 * in_to_m}"/>
   <xacro:property name="lidar_z_offset" value="${4.62 * in_to_m}"/>
-  <xacro:property name="gps_x_offset" value="${tower_x_offset}"/>
+  <xacro:property name="gps_x_offset" value="${0}"/>
+  <xacro:property name="gps_y_offset" value="${(tower_width / 2) - gps_radius}"/>
   <xacro:property name="gps_z_offset" value="${(tower_height / 2) + (gps_height / 2)}"/>
   <xacro:property name="camera_x_offset" value="${(tower_length / 2) + (2 * in_to_m)}"/>

File: ora_description/description/sensors.xacro (robot description, xacro)
@@ -158,5 +158,5 @@
     <parent link="tower_link"/>
     <child link="gnss_link"/>
-    <origin xyz="0 0 ${gps_z_offset}" rpy="0 0 0"/>
+    <origin xyz="${gps_x_offset} ${gps_y_offset} ${gps_z_offset}" rpy="0 0 0"/>
   </joint>
   <!-- <gazebo reference="gnss_link">

Commit message: move imu

File: ora_description/description/dimensions.xacro (robot description, xacro)
@@ -64,4 +64,4 @@
   <xacro:property name="camera_x_offset" value="${(tower_length / 2) + (2 * in_to_m)}"/>
   <xacro:property name="camera_z_offset" value="${(tower_height / 2)}"/>
-  <xacro:property name="imu_z_offset" value="${base_z_offset + (base_height / 2) - (0.25 * in_to_m)}"/>
+  <xacro:property name="imu_z_offset" value="${base_z_offset - (base_height / 2) + (9 * in_to_m)}"/>
 </robot>

Commit message: 13

File: ora_description/description/dimensions.xacro (robot description, xacro)
@@ -19,5 +19,5 @@
   <xacro:property name="tower_height" value="${26.25 * in_to_m}"/>
   <!-- Wheel Dimensions / Location -->
-  <xacro:property name="main_wheel_diameter" value="${11.97 * in_to_m}"/>
+  <xacro:property name="main_wheel_diameter" value="${13 * in_to_m}"/>
   <xacro:property name="main_wheel_radius" value="${main_wheel_diameter / 2}"/>
   <xacro:property name="main_wheel_width" value="${48 * mm_to_m}"/>
