Commit message: Add placeholder for real control

File: ora_description/description/anteater.urdf.xacro (robot description, xacro)
@@ -1,7 +1,4 @@
 <?xml version="1.0"?>
 <robot xmlns:xacro="https://www.ros.org/wiki/xacro" name="robot_name">
-  <!-- Args -->
-  <!-- General -->
-  <xacro:arg name="sim_mode" default="false"/>
   <!-- Include all of the pieces of the robot -->
   <xacro:include filename="anteater_core.xacro"/>

File: ora_description/description/ros2_control.xacro (robot description, xacro)
@@ -1,49 +1,56 @@
 <?xml version="1.0"?>
 <robot xmlns:xacro="https://www.ros.org/wiki/xacro">
-  <ros2_control name="GazeboSystem" type="system">
-    <hardware>
-      <plugin>gz_ros2_control/GazeboSimSystem</plugin>
-    </hardware>
-    <!-- Main Wheel Joints -->
-    <joint name="left_wheel_joint">
-      <command_interface name="velocity">
+  <!-- Args -->
+  <xacro:arg name="sim_mode" default="true"/>
+  <xacro:if value="$(arg sim_mode)">
+    <ros2_control name="GazeboSystem" type="system">
+      <hardware>
+        <plugin>gz_ros2_control/GazeboSimSystem</plugin>
+      </hardware>
+      <!-- Main Wheel Joints -->
+      <joint name="left_wheel_joint">
+        <command_interface name="velocity">
+            <param name="min">-10</param>
+            <param name="max">10</param>
+        </command_interface>
+        <state_interface name="position"/>
+        <state_interface name="velocity"/>
+      </joint>
+      <joint name="right_wheel_joint">
+        <command_interface name="velocity">
           <param name="min">-10</param>
           <param name="max">10</param>
-      </command_interface>
-      <state_interface name="position"/>
-      <state_interface name="velocity"/>
-    </joint>
-    <joint name="right_wheel_joint">
-      <command_interface name="velocity">
-        <param name="min">-10</param>
-        <param name="max">10</param>
-      </command_interface>
-      <state_interface name="position"/>
-      <state_interface name="velocity"/>
-    </joint>
-    <!-- Caster Joints -->
-    <joint name="left_front_caster_joint">
-      <state_interface name="position"/>
-      <state_interface name="velocity"/>
-    </joint>
-    <joint name="right_front_caster_joint">
-      <state_interface name="position"/>
-      <state_interface name="velocity"/>
-    </joint>
-    <joint name="left_back_caster_joint">
-      <state_interface name="position"/>
-      <state_interface name="velocity"/>
-    </joint>
-    <joint name="right_back_caster_joint">
-      <state_interface name="position"/>
-      <state_interface name="velocity"/>
-    </joint>
-  </ros2_control>
-  <gazebo>
-    <plugin name="gz_ros2_control::GazeboSimROS2ControlPlugin" filename="libgz_ros2_control-system.so">
-      <robot_param>robot_description</robot_param>
-      <robot_param_node>robot_state_publisher</robot_param_node>
-      <parameters>$(find ora_sim)/config/sim_controller.yaml</parameters>
-    </plugin>
-  </gazebo>
+        </command_interface>
+        <state_interface name="position"/>
+        <state_interface name="velocity"/>
+      </joint>
+      <!-- Caster Joints -->
+      <joint name="left_front_caster_joint">
+        <state_interface name="position"/>
+        <state_interface name="velocity"/>
+      </joint>
+      <joint name="right_front_caster_joint">
+        <state_interface name="position"/>
+        <state_interface name="velocity"/>
+      </joint>
+      <joint name="left_back_caster_joint">
+        <state_interface name="position"/>
+        <state_interface name="velocity"/>
+      </joint>
+      <joint name="right_back_caster_joint">
+        <state_interface name="position"/>
+        <state_interface name="velocity"/>
+      </joint>
+    </ros2_control>
+    <gazebo>
+      <plugin name="gz_ros2_control::GazeboSimROS2ControlPlugin" filename="libgz_ros2_control-system.so">
+        <robot_param>robot_description</robot_param>
+        <robot_param_node>robot_state_publisher</robot_param_node>
+        <parameters>$(find ora_sim)/config/sim_controller.yaml</parameters>
+      </plugin>
+    </gazebo>
+  </xacro:if>
+  <xacro:unless value="$(arg sim_mode)">
+    <!-- TODO: Add real hardware control -->
+  </xacro:unless>
 </robot>

Commit message: couple o fixes

File: ora_description/description/anteater.urdf.xacro (robot description, xacro)
@@ -1,4 +1,4 @@
 <?xml version="1.0"?>
-<robot xmlns:xacro="https://www.ros.org/wiki/xacro" name="robot_name">
+<robot xmlns:xacro="https://www.ros.org/wiki/xacro" name="erdferkel">
   <xacro:arg name="sim_mode" default="false"/>
   <!-- Include all of the pieces of the robot -->

File: ora_description/description/anteater_core.xacro (robot description, xacro)
@@ -31,5 +31,5 @@
     </visual>
     <collision>
-      <origin xyz="${0 + (back_caster_x_offset / 4)} 0 ${back_caster_radius / 4}" rpy="0 0 0"/>
+      <origin xyz="${base_x_offset} 0 ${base_z_offset}" rpy="0 0 0"/>
       <geometry>
         <box size="${base_length} ${base_width} ${base_height}"/>
@@ -37,5 +37,5 @@
     </collision>
     <xacro:inertial_box mass="50.0" x="${base_length}" y="${base_width}" z="${base_height}">
-      <origin xyz="0 0 0" rpy="0 0 0"/>
+      <origin xyz="${base_x_offset} 0 ${base_z_offset}" rpy="0 0 0"/>
     </xacro:inertial_box>
   </link>

Commit message: add zed 2i to urdf

File: ora_description/description/anteater.urdf.xacro (robot description, xacro)
@@ -8,3 +8,4 @@
   <xacro:include filename="sensors.xacro"/>
   <xacro:include filename="ros2_control.xacro"/>
+  <xacro:include filename="camera.xacro"/>
 </robot>

File: ora_description/description/dimensions.xacro (robot description, xacro)
@@ -48,4 +48,5 @@
   <xacro:property name="camera_width" value="0.130"/>
   <xacro:property name="camera_height" value="0.022"/>
+  <xacro:property name="zed2i_height" value="${30.25 * mm_to_m}"/>
   <!-- IMU Dimensions -->
   <xacro:property name="imu_length" value="${25 * mm_to_m}"/>

File: ora_description/description/sensors.xacro (robot description, xacro)
@@ -71,35 +71,4 @@
     </sensor>
   </gazebo>
-  <!-- Simulated RGBD Camera -->
-  <link name="camera_link">
-    <visual>
-      <origin xyz="0 0 0" rpy="0 0 0"/>
-      <geometry>
-        <box size="${camera_length} ${camera_width} ${camera_height}"/>
-      </geometry>
-      <material name="yellow"/>
-    </visual>
-    <collision>
-      <origin xyz="0 0 0" rpy="0 0 0"/>
-      <geometry>
-        <box size="${camera_length} ${camera_width} ${camera_height}"/>
-      </geometry>
-    </collision>
-    <xacro:inertial_box mass="0.035" x="${camera_length}" y="${camera_width}" z="${camera_height}">
-      <origin xyz="0 0 0" rpy="0 0 0"/>
-    </xacro:inertial_box>
-  </link>
-  <joint name="camera_joint" type="fixed">
-    <parent link="tower_link"/>
-    <child link="camera_link"/>
-    <origin xyz="${camera_x_offset} 0 ${camera_z_offset}" rpy="0 0.610865 0"/>
-  </joint>
-  <!-- For use with the line detection -->
-  <link name='camera_link_optical' />
-  <joint name="camera_optical_joint" type="fixed">
-    <parent link="camera_link"/>
-    <child link="camera_link_optical"/>
-    <origin xyz="0 0 0" rpy="-1.57079632679 0 -1.57079632679"/>
-  </joint>
   <!-- Simulated RGBD camera plugin -->
   <gazebo reference="camera_link">
