Commit message: Added camera module

File: ora_description/description/sensors.xacro (robot description, xacro)
@@ -1,4 +1,4 @@
 <?xml version="1.0"?>
-<robot xmlns:xacro="https://www.ros.org/wiki/xacro">
+<robot xmlns:xacro="http://www.ros.org/wiki/xacro">
   <xacro:include filename="dimensions.xacro"/>
   <xacro:include filename="inertia_macros.xacro"/>
@@ -28,5 +28,5 @@
     <origin xyz="${lidar_x_offset} 0 ${lidar_z_offset}" rpy="0 0 0"/>
   </joint>
-  <!-- Lidar Plugin -->
+  <!-- Lidar Gazebo plugin -->
   <gazebo reference="lidar_link">
     <sensor name="lidar" type="gpu_lidar">
@@ -90,5 +90,5 @@
     <origin xyz="0 0 0.01" rpy="0 0 0"/>
   </joint>
-  <!-- IMU Plugin -->
+  <!-- IMU Gazebo plugin -->
   <gazebo reference="imu_link">
     <sensor name="imu_sensor" type="imu">
@@ -100,81 +100,88 @@
       <imu>
         <angular_velocity>
-          <x>
-            <noise type="gaussian">
-              <mean>0.0</mean>
-              <stddev>2e-4</stddev>
-              <bias_mean>0.0000075</bias_mean>
-              <bias_stddev>0.0000008</bias_stddev>
-            </noise>
-          </x>
-          <y>
-            <noise type="gaussian">
-              <mean>0.0</mean>
-              <stddev>2e-4</stddev>
-              <bias_mean>0.0000075</bias_mean>
-              <bias_stddev>0.0000008</bias_stddev>
-            </noise>
-          </y>
-          <z>
-            <noise type="gaussian">
-                <mean>0.0</mean>
-                <stddev>2e-4</stddev>
-                <bias_mean>0.0000075</bias_mean>
-                <bias_stddev>0.0000008</bias_stddev>
-            </noise>
-          </z>
+          <x><noise type="gaussian"><mean>0.0</mean><stddev>2e-4</stddev><bias_mean>0.0000075</bias_mean><bias_stddev>0.0000008</bias_stddev></noise></x>
+          <y><noise type="gaussian"><mean>0.0</mean><stddev>2e-4</stddev><bias_mean>0.0000075</bias_mean><bias_stddev>0.0000008</bias_stddev></noise></y>
+          <z><noise type="gaussian"><mean>0.0</mean><stddev>2e-4</stddev><bias_mean>0.0000075</bias_mean><bias_stddev>0.0000008</bias_stddev></noise></z>
         </angular_velocity>
-      <linear_acceleration>
-          <x>
-            <noise type="gaussian">
-                <mean>0.0</mean>
-                <stddev>1.7e-2</stddev>
-                <bias_mean>0.1</bias_mean>
-                <bias_stddev>0.001</bias_stddev>
-            </noise>
-          </x>
-          <y>
-            <noise type="gaussian">
-                <mean>0.0</mean>
-                <stddev>1.7e-2</stddev>
-                <bias_mean>0.1</bias_mean>
-                <bias_stddev>0.001</bias_stddev>
-            </noise>
-          </y>
-          <z>
-            <noise type="gaussian">
-                <mean>0.0</mean>
-                <stddev>1.7e-2</stddev>
-                <bias_mean>0.1</bias_mean>
-                <bias_stddev>0.001</bias_stddev>
-            </noise>
-          </z>
+        <linear_acceleration>
+          <x><noise type="gaussian"><mean>0.0</mean><stddev>1.7e-2</stddev><bias_mean>0.1</bias_mean><bias_stddev>0.001</bias_stddev></noise></x>
+          <y><noise type="gaussian"><mean>0.0</mean><stddev>1.7e-2</stddev><bias_mean>0.1</bias_mean><bias_stddev>0.001</bias_stddev></noise></y>
+          <z><noise type="gaussian"><mean>0.0</mean><stddev>1.7e-2</stddev><bias_mean>0.1</bias_mean><bias_stddev>0.001</bias_stddev></noise></z>
         </linear_acceleration>
       </imu>
     </sensor>
   </gazebo>
-  <gazebo>
-    <plugin filename="gz-sim-diff-drive-system" name="gz::sim::systems::DiffDrive">
-      <!-- wheels -->
-      <left_joint>left_wheel_joint</left_joint>
-      <right_joint>right_wheel_joint</right_joint>
-      <!-- kinematics -->
-      <wheel_separation>${base_width}</wheel_separation>
-      <wheel_radius>${main_wheel_radius}</wheel_radius>
-      <!-- limits -->
-      <max_linear_acceleration>2.0</max_linear_acceleration>
-      <!-- input -->
-      <topic>/demo/cmd_vel</topic>
-      <!-- output -->
-      <odom_topic>/demo/odom</odom_topic>
-      <tf_topic>/tf</tf_topic>
-      <frame_id>odom</frame_id>
-      <child_frame_id>base_link</child_frame_id>
-    </plugin>
-    <plugin
-      filename="gz-sim-joint-state-publisher-system"
-      name="gz::sim::systems::JointStatePublisher">
-      <topic>joint_states</topic>
-    </plugin>
+  <!-- USB Camera -->
+  <link name="camera_link">
+    <inertial>
+      <origin xyz="0 0 0" rpy="0 0 0"/>
+      <mass value="0.05"/>
+      <inertia ixx="0.0001" ixy="0" ixz="0" iyy="0.0001" iyz="0" izz="0.0001"/>
+    </inertial>
+    <visual>
+      <origin xyz="0 0 0" rpy="0 0 0"/>
+      <geometry>
+        <box size="0.04 0.10 0.04"/>  <!-- slightly larger for better visibility in RViz/Gazebo -->
+      </geometry>
+      <material name="black"/>
+    </visual>
+    <collision>
+      <origin xyz="0 0 0" rpy="0 0 0"/>
+      <geometry>
+        <box size="0.04 0.10 0.04"/>
+      </geometry>
+    </collision>
+  </link>
+  <joint name="camera_joint" type="fixed">
+    <parent link="base_link"/>
+    <child link="camera_link"/>
+    <!-- Suggested position: forward 20 cm, up 25 cm – adjust based on real mounting -->
+    <origin xyz="0.20 0.0 0.25" rpy="0 0 0"/>
+  </joint>
+  <!-- Optical frame (ROS standard: z forward, x right, y down) -->
+  <link name="camera_optical_frame"/>
+  <joint name="camera_optical_joint" type="fixed">
+    <parent link="camera_link"/>
+    <child link="camera_optical_frame"/>
+    <origin xyz="0 0 0" rpy="${-pi/2} 0 ${-pi/2}"/>
+  </joint>
+  <!-- Gazebo camera plugin (for simulation – matches real usb_cam topics) -->
+  <gazebo reference="camera_link">
+    <sensor name="ora_usb_camera" type="camera">
+      <always_on>true</always_on>
+      <visualize>true</visualize>
+      <update_rate>30.0</update_rate>
+      <camera>
+        <horizontal_fov>1.047</horizontal_fov>  <!-- ≈60 deg FOV – common for USB cams; adjust if known -->
+        <image>
+          <width>640</width>
+          <height>480</height>
+          <format>R8G8B8</format>
+        </image>
+        <clip>
+          <near>0.05</near>
+          <far>100</far>
+        </clip>
+      </camera>
+      <plugin name="ora_camera_plugin" filename="libgazebo_ros_camera.so">
+        <ros>
+          <namespace>/ora_camera</namespace>
+          <remapping>image_raw:=image_raw</remapping>
+          <remapping>camera_info:=camera_info</remapping>
+        </ros>
+        <cameraName>ora_camera</cameraName>
+        <imageTopicName>image_raw</imageTopicName>
+        <cameraInfoTopicName>camera_info</cameraInfoTopicName>
+        <frameName>camera_optical_frame</frameName>
+        <alwaysOn>true</alwaysOn>
+        <updateRate>0.0</updateRate>
+        <!-- Optional distortion (set to 0 if no calibration yet) -->
+        <distortionK1>0.0</distortionK1>
+        <distortionK2>0.0</distortionK2>
+        <distortionK3>0.0</distortionK3>
+        <distortionT1>0.0</distortionT1>
+        <distortionT2>0.0</distortionT2>
+      </plugin>
+    </sensor>
   </gazebo>
 </robot>

Commit message: feat: Add RGBD camera package.

File: ora_description/description/sensors.xacro (robot description, xacro)
@@ -65,4 +65,38 @@
     </sensor>
   </gazebo>
+  <!-- RGBD Camera -->
+  <link name="camera_link">
+    <visual>
+      <geometry>
+        <box size="0.05 0.05 0.05"/>
+      </geometry>
+    </visual>
+  </link>
+  <joint name="camera_joint" type="fixed">
+    <parent link="base_link"/>
+    <child link="camera_link"/>
+    <origin xyz="0.2 0 0.3" rpy="0 0 0"/>
+  </joint>
+  <gazebo reference="camera_link">
+    <sensor name="rgbd_camera" type="rgbd_camera">
+      <camera>
+        <horizontal_fov>1.2</horizontal_fov>
+        <image>
+          <width>640</width>
+          <height>480</height>
+        </image>
+        <clip>
+          <near>0.1</near>
+          <far>10.0</far>
+        </clip>
+        <optical_frame_id>camera_link_optical</optical_frame_id>
+      </camera>
+      <always_on>true</always_on>
+      <update_rate>30</update_rate>
+      <visualize>true</visualize>
+      <topic>rgbd_camera</topic>
+      <gz_frame_id>camera_link</gz_frame_id>
+    </sensor>
+  </gazebo>
   <!-- GPS -->
   <link name="gps_link">

Commit message: fix: Use nav2 depth camera and fix implementation.

File: ora_description/description/sensors.xacro (robot description, xacro)
@@ -68,18 +68,35 @@
   <link name="camera_link">
     <visual>
-      <geometry>
-        <box size="0.05 0.05 0.05"/>
-      </geometry>
-    </visual>
+      <origin xyz="0 0 0" rpy="0 0 0"/>
+      <geometry>
+        <box size="0.015 0.130 0.022"/>
+      </geometry>
+    </visual>
+    <collision>
+      <origin xyz="0 0 0" rpy="0 0 0"/>
+      <geometry>
+        <box size="0.015 0.130 0.022"/>
+      </geometry>
+    </collision>
+    <inertial>
+      <origin xyz="0 0 0" rpy="0 0 0"/>
+      <mass value="0.035"/>
+      <inertia ixx="0.001" ixy="0" ixz="0" iyy="0.001" iyz="0" izz="0.001" />
+    </inertial>
   </link>
   <joint name="camera_joint" type="fixed">
     <parent link="base_link"/>
     <child link="camera_link"/>
-    <origin xyz="0.2 0 0.3" rpy="0 0 0"/>
+    <origin xyz="0.45 0 0.4" rpy="0 0 0"/>
   </joint>
   <gazebo reference="camera_link">
-    <sensor name="rgbd_camera" type="rgbd_camera">
+    <sensor name="depth_camera" type="rgbd_camera">
+      <always_on>true</always_on>
+      <visualize>true</visualize>
+      <update_rate>5.0</update_rate>
+      <topic>depth_camera</topic>
+      <gz_frame_id>camera_link</gz_frame_id>
       <camera>
-        <horizontal_fov>1.2</horizontal_fov>
+        <horizontal_fov>1.047198</horizontal_fov>
         <image>
           <width>640</width>
@@ -87,14 +104,21 @@
         </image>
         <clip>
-          <near>0.1</near>
-          <far>10.0</far>
+          <near>0.05</near>
+          <far>3</far>
         </clip>
-        <optical_frame_id>camera_link_optical</optical_frame_id>
       </camera>
-      <always_on>true</always_on>
-      <update_rate>30</update_rate>
-      <visualize>true</visualize>
-      <topic>rgbd_camera</topic>
-      <gz_frame_id>camera_link</gz_frame_id>
+      <baseline>0.2</baseline>
+      <pointCloudCutoff>0.5</pointCloudCutoff>
+      <pointCloudCutoffMax>3.0</pointCloudCutoffMax>
+      <distortionK1>0</distortionK1>
+      <distortionK2>0</distortionK2>
+      <distortionK3>0</distortionK3>
+      <distortionT1>0</distortionT1>
+      <distortionT2>0</distortionT2>
+      <CxPrime>0</CxPrime>
+      <Cx>0</Cx>
+      <Cy>0</Cy>
+      <focalLength>0</focalLength>
+      <hackBaseline>0</hackBaseline>
     </sensor>
   </gazebo>

Commit message: feat: Add dark_gray color to previously uncolored sensor components.

File: ora_description/description/sensors.xacro (robot description, xacro)
@@ -21,4 +21,5 @@
         <cylinder radius="${lidar_radius}" length="${lidar_height}"/>
       </geometry>
+      <material name="dark_gray"/>
     </visual>
   </link>
@@ -83,4 +84,5 @@
         <cylinder radius="${gps_radius}" length="${gps_height}"/>
       </geometry>
+      <material name="dark_gray"/>
     </visual>
   </link>
@@ -126,4 +128,5 @@
         <box size="0.1 0.1 0.1"/>
       </geometry>
+      <material name="dark_gray"/>
     </visual>
     <collision>

Commit message: feat: Add simulated rgbd camera plugin.

File: ora_description/description/sensors.xacro (robot description, xacro)
@@ -66,4 +66,64 @@
     </sensor>
   </gazebo>
+  <!-- Simulated RGBD Camera -->
+  <link name="camera_link">
+    <visual>
+      <origin xyz="0 0 0" rpy="0 0 0"/>
+      <geometry>
+        <box size="0.015 0.130 0.022"/>
+      </geometry>
+      <material name="dark_gray"/>
+    </visual>
+    <collision>
+      <origin xyz="0 0 0" rpy="0 0 0"/>
+      <geometry>
+        <box size="0.015 0.130 0.022"/>
+      </geometry>
+    </collision>
+    <inertial>
+      <origin xyz="0 0 0" rpy="0 0 0"/>
+      <mass value="0.035"/>
+      <inertia ixx="0.001" ixy="0" ixz="0" iyy="0.001" iyz="0" izz="0.001" />
+    </inertial>
+  </link>
+  <joint name="camera_joint" type="fixed">
+    <parent link="base_link"/>
+    <child link="camera_link"/>
+    <origin xyz="0.2 0 0.4" rpy="0 0 0"/>
+  </joint>
+  <!-- Simulated RGBD camera plugin -->
+  <gazebo reference="camera_link">
+    <sensor name="depth_camera" type="rgbd_camera">
+      <always_on>true</always_on>
+      <visualize>true</visualize>
+      <update_rate>5.0</update_rate>
+      <topic>depth_camera</topic>
+      <gz_frame_id>camera_link</gz_frame_id>
+      <camera>
+        <horizontal_fov>1.047198</horizontal_fov>
+        <image>
+          <width>640</width>
+          <height>480</height>
+        </image>
+        <clip>
+          <near>0.05</near>
+          <far>3</far>
+        </clip>
+      </camera>
+      <baseline>0.2</baseline>
+      <pointCloudCutoff>0.5</pointCloudCutoff>
+      <pointCloudCutoffMax>3.0</pointCloudCutoffMax>
+      <distortionK1>0</distortionK1>
+      <distortionK2>0</distortionK2>
+      <distortionK3>0</distortionK3>
+      <distortionT1>0</distortionT1>
+      <distortionT2>0</distortionT2>
+      <CxPrime>0</CxPrime>
+      <Cx>0</Cx>
+      <Cy>0</Cy>
+      <focalLength>0</focalLength>
+      <hackBaseline>0</hackBaseline>
+    </sensor>
+  </gazebo>
   <!-- GPS -->
   <link name="gps_link">

Commit message: Fix mutli-publisher simulation issues

File: ora_description/description/sensors.xacro (robot description, xacro)
@@ -127,5 +127,5 @@
   </gazebo>
   <!-- GPS -->
-  <link name="gps_link">
+  <link name="gnss_link">
     <inertial>
       <origin xyz="0 0 0" rpy="0 0 0"/>
@@ -149,13 +149,13 @@
   <joint name="gps_joint" type="fixed">
     <parent link="base_link"/>
-    <child link="gps_link"/>
+    <child link="gnss_link"/>
     <origin xyz="${gps_x_offset} 0 ${gps_z_offset}" rpy="0 0 0"/>
   </joint>
-  <gazebo reference="gps_link">
+  <gazebo reference="gnss_link">
     <sensor name="navsat" type="navsat">
       <always_on>true</always_on>
       <update_rate>8</update_rate>
       <topic>/gnss/fix</topic>
-      <gz_frame_id>gps_link</gz_frame_id>
+      <gz_frame_id>gnss_link</gz_frame_id>
       <navsat>
         <position_sensing>

Commit message: Update URDF (#60)
* updated robot's dimensions

* add sesnor tower

* couple o fixes

* update sensors to real positions

* update IMU to real

* update footprint

* Adjust GPS offset

* move imu

* 13

* add zed 2i to urdf

---------

Co-authored-by: ZacharyLain <zacharytlain@gmail.com>

File: ora_description/description/sensors.xacro (robot description, xacro)
@@ -5,9 +5,7 @@
   <!-- Lidar -->
   <link name="lidar_link">
-    <inertial>
-      <origin xyz="0 0 0" rpy="0 0 0"/>
-      <mass value="0.125"/>
-      <inertia ixx="0.001" ixy="0" ixz="0" iyy="0.001" iyz="0" izz="0.001" />
-    </inertial>
+    <xacro:inertial_cylinder mass="0.125" length="${lidar_height}" radius="${lidar_radius}">
+      <origin xyz="0 0 0" rpy="0 0 0"/>
+    </xacro:inertial_cylinder>
     <collision>
       <origin xyz="0 0 0" rpy="0 0 0"/>
@@ -21,5 +19,5 @@
         <cylinder radius="${lidar_radius}" length="${lidar_height}"/>
       </geometry>
-      <material name="dark_gray"/>
+      <material name="blue"/>
     </visual>
   </link>
@@ -29,4 +27,11 @@
     <origin xyz="${lidar_x_offset} 0 ${lidar_z_offset}" rpy="0 0 0"/>
   </joint>
+  <xacro:unless value="$(arg sim_mode)">
+    <joint name="velodyne_joint" type="fixed">
+      <parent link="lidar_link"/>
+      <child link="velodyne"/>
+      <origin xyz="0 0 0" rpy="0 0 0"/>
+    </joint>
+  </xacro:unless>
   <!-- Lidar Plugin -->
   <gazebo reference="lidar_link">
@@ -66,37 +71,4 @@
     </sensor>
   </gazebo>
-  <!-- Simulated RGBD Camera -->
-  <link name="camera_link">
-    <visual>
-      <origin xyz="0 0 0" rpy="0 0 0"/>
-      <geometry>
-        <box size="0.015 0.130 0.022"/>
-      </geometry>
-      <material name="dark_gray"/>
-    </visual>
-    <collision>
-      <origin xyz="0 0 0" rpy="0 0 0"/>
-      <geometry>
-        <box size="0.015 0.130 0.022"/>
-      </geometry>
-    </collision>
-    <inertial>
-      <origin xyz="0 0 0" rpy="0 0 0"/>
-      <mass value="0.035"/>
-      <inertia ixx="0.001" ixy="0" ixz="0" iyy="0.001" iyz="0" izz="0.001" />
-    </inertial>
-  </link>
-  <joint name="camera_joint" type="fixed">
-    <parent link="base_link"/>
-    <child link="camera_link"/>
-    <origin xyz="0.2 0 0.4" rpy="0 0 0"/>
-  </joint>
-  <!-- For use with the line detection -->
-  <link name='camera_link_optical' />
-  <joint name="camera_optical_joint" type="fixed">
-    <parent link="camera_link"/>
-    <child link="camera_link_optical"/>
-    <origin xyz="0 0 0" rpy="-1.57079632679 0 -1.57079632679"/>
-  </joint>
   <!-- Simulated RGBD camera plugin -->
   <gazebo reference="camera_link">
@@ -135,9 +107,7 @@
   <!-- GPS -->
   <link name="gnss_link">
-    <inertial>
-      <origin xyz="0 0 0" rpy="0 0 0"/>
-      <mass value="0.125"/>
-      <inertia ixx="0.001" ixy="0" ixz="0" iyy="0.001" iyz="0" izz="0.001" />
-    </inertial>
+    <xacro:inertial_cylinder mass="0.125" length="${gps_height}" radius="${gps_radius}">
+      <origin xyz="0 0 0" rpy="0 0 0"/>
+    </xacro:inertial_cylinder>
     <collision>
       <origin xyz="0 0 0" rpy="0 0 0"/>
@@ -151,11 +121,11 @@
         <cylinder radius="${gps_radius}" length="${gps_height}"/>
       </geometry>
-      <material name="dark_gray"/>
+      <material name="red"/>
     </visual>
   </link>
   <joint name="gps_joint" type="fixed">
-    <parent link="base_link"/>
+    <parent link="tower_link"/>
     <child link="gnss_link"/>
-    <origin xyz="${gps_x_offset} 0 ${gps_z_offset}" rpy="0 0 0"/>
+    <origin xyz="${gps_x_offset} ${gps_y_offset} ${gps_z_offset}" rpy="0 0 0"/>
   </joint>
   <!-- <gazebo reference="gnss_link">
@@ -185,20 +155,18 @@
   <!-- IMU -->
   <link name="imu_link">
-    <inertial>
-      <origin xyz="0 0 0" rpy="0 0 0"/>
-      <mass value="0.1"/>
-      <inertia ixx="0.0001" ixy="0" ixz="0" iyy="0.0001" iyz="0" izz="0.0001"/>
-    </inertial>
+    <xacro:inertial_box mass="0.01" x="${imu_length}" y="${imu_width}" z="${imu_height}">
+      <origin xyz="0 0 0" rpy="0 0 0"/>
+    </xacro:inertial_box>
     <visual>
       <origin xyz="0 0 0" rpy="0 0 0"/>
       <geometry>
-        <box size="0.1 0.1 0.1"/>
-      </geometry>
-      <material name="dark_gray"/>
+        <box size="${imu_length} ${imu_width} ${imu_height}"/>
+      </geometry>
+      <material name="purple"/>
     </visual>
     <collision>
       <origin xyz="0 0 0" rpy="0 0 0"/>
       <geometry>
-        <box size="0.1 0.1 0.1"/>
+        <box size="${imu_length} ${imu_width} ${imu_height}"/>
       </geometry>
     </collision>
@@ -207,5 +175,5 @@
     <parent link="base_link"/>
     <child link="imu_link"/>
-    <origin xyz="0 0 0.01" rpy="0 0 0"/>
+    <origin xyz="0 0 ${imu_z_offset}" rpy="0 0 0"/>
   </joint>
   <!-- IMU Plugin -->

Commit message: Lidar launch

File: ora_description/description/sensors.xacro (robot description, xacro)
@@ -28,4 +28,5 @@
   </joint>
   <xacro:unless value="$(arg sim_mode)">
+    <link name="velodyne" />
     <joint name="velodyne_joint" type="fixed">
       <parent link="lidar_link"/>
